Commit message: Sensor de Contacto

File: p_gmota_description/urdf/p_gmota.gazebo.xacro (robot description, xacro)
@@ -167,3 +167,17 @@
     </sensor>
   </gazebo>
+  <!-- Contact Sensor -->
+  <gazebo reference="base_link">
+    <sensor name="base_link" type="contact">
+      <update_rate>1000.0</update_rate>
+      <always_on>true</always_on>
+      <contact>
+        <collision> "base_footprint_fixed_joint_lump__base_link_collision" </collision>
+      </contact>
+      <plugin name="base_link_contact_sensor_plugin" filename="libgazebo_ros_bumper.so">
+        <bumperTopicName>contact</bumperTopicName>
+        <frameName>world</frameName>
+      </plugin>
+    </sensor>
+  </gazebo>
 </robot>

Commit message: Sensor de Contacto

File: p_gmota_description/urdf/p_gmota.gazebo.xacro (robot description, xacro)
@@ -173,5 +173,5 @@
       <always_on>true</always_on>
       <contact>
-        <collision> "base_footprint_fixed_joint_lump__base_link_collision" </collision>
+        <collision> base_footprint_fixed_joint_lump__base_link_collision </collision>
       </contact>
       <plugin name="base_link_contact_sensor_plugin" filename="libgazebo_ros_bumper.so">
